File: DST.kicad_pcb (KiCad board)
At the start: 6 copper layers, 158.5 x 83.3 mm, 285 parts, among them J1 1727010, J13 DC-005-5A-2.0, J14 1981568-1, J18 825434-5, J19 825434-5, J2 5-146280-3, J20 825434-5, J21 825434-5, J22 825434-5, J23 825434-5, J24 825434-5, J25 825434-5, J26 825434-5, J27 825434-5, J28 825434-5, J29 825434-5, J3 20021121-00020C4LF, SW1 SW_Push, SW2 SW_Push, SW3 219-3LPSTR, U1 RP2350B-QFN80, U10 DRIVER-A4988SETTR-T_QFN28_, U11 DRIVER-A4988SETTR-T_QFN28_, U12 DRIVER-A4988SETTR-T_QFN28_, U13 DRIVER-A4988SETTR-T_QFN28_, U14 DRIVER-A4988SETTR-T_QFN28_, U15 DRIVER-A4988SETTR-T_QFN28_, U16 PMIC-AP1509-SG-13_SOIC8_, U2 ABM8-272-T3, U3 W25Q128JVSIQ, U4 DRIVER-A4988SETTR-T_QFN28_, U5 DRIVER-A4988SETTR-T_QFN28_, U6 DRIVER-A4988SETTR-T_QFN28_, U7 DRIVER-A4988SETTR-T_QFN28_, U8 DRIVER-A4988SETTR-T_QFN28_, U9 DRIVER-A4988SETTR-T_QFN28_

Commit message: newsest changes
Parts:
- removed D5, D7: 5988170107F, 5988170107F:LEDC2012X70N
- removed J18, J19, J20, J21, J22, J23, J24, J25, J26, J27, J28, J29: 825434-5, 825434-5:TE_825434-5
- removed SW3: 219-3LPSTR, 219-3LPSTR:SW_219-3LPSTR
- added J10: 77311-462K05LF, 77311-462K05LF:HDRV5W62P0X254_1X5_1270X240X1624P, F.Cu at (181.6, 131.4)
- added J11: 77311-462K05LF, 77311-462K05LF:HDRV5W62P0X254_1X5_1270X240X1624P, F.Cu at (162.4, 51.4)
- added J12: 77311-462K05LF, 77311-462K05LF:HDRV5W62P0X254_1X5_1270X240X1624P, F.Cu at (203.0, 130.9)
- added J15: 77311-462K05LF, 77311-462K05LF:HDRV5W62P0X254_1X5_1270X240X1624P, F.Cu at (139.1, 51.4)
- added J16: 77311-462K05LF, 77311-462K05LF:HDRV5W62P0X254_1X5_1270X240X1624P, F.Cu at (226.3, 131.4)
- added J17: 77311-462K05LF, 77311-462K05LF:HDRV5W62P0X254_1X5_1270X240X1624P, F.Cu at (112.9, 51.4)
- added J4: 77311-462K05LF, 77311-462K05LF:HDRV5W62P0X254_1X5_1270X240X1624P, F.Cu at (110.4, 131.4)
- added J5: 77311-462K05LF, 77311-462K05LF:HDRV5W62P0X254_1X5_1270X240X1624P, F.Cu at (233.5, 51.4)
- added J6: 77311-462K05LF, 77311-462K05LF:HDRV5W62P0X254_1X5_1270X240X1624P, F.Cu at (134.2, 131.4)
- added J7: 77311-462K05LF, 77311-462K05LF:HDRV5W62P0X254_1X5_1270X240X1624P, F.Cu at (210.2, 51.4)
- added J8: 77311-462K05LF, 77311-462K05LF:HDRV5W62P0X254_1X5_1270X240X1624P, F.Cu at (159.2, 131.4)
- added J9: 77311-462K05LF, 77311-462K05LF:HDRV5W62P0X254_1X5_1270X240X1624P, F.Cu at (186.6, 51.4)
- added LED1: 150080GS75000, KiCad:LEDM2012X80N, F.Cu at (110.2, 83.6)
- added LED2: 150080GS75000, KiCad:LEDM2012X80N, F.Cu at (246.1, 106.5)
- added S2: 1MS3T1B1M2QES, 1MS3T1B1M2QES:1MS3T1B1M2QES, F.Cu at (226.9, 93.3)
- S1: value 100SP1T2B4M7QE -> NDS-03V; footprint 100SP1T2B4M7QE:SW_100SP1T2B4M7QE -> NDS-03V:NDS03V
- moved S1 66.3 mm to (162.4, 78.6), turned to -90 degrees
- moved R98 9.50 mm to (133.9, 70.8)
- moved R81 9.45 mm to (180.0, 70.7)
- moved R106 9.39 mm to (107.0, 70.9)
- moved R22 9.37 mm to (163.1, 110.0)
- moved R38 9.37 mm to (207.6, 110.2)
- moved R54 9.32 mm to (227.2, 70.5)
- moved R90 9.27 mm to (157.2, 70.4)
- moved R62 9.17 mm to (202.9, 70.3)
- moved R14 9.11 mm to (139.0, 110.3)
- moved R46 9.07 mm to (231.0, 110.7)
- moved R13 9.07 mm to (115.5, 110.8)
- moved R30 8.99 mm to (185.7, 110.0)
- moved R94 2.75 mm to (234.5, 110.8), turned to 180 degrees
- moved R66 2.62 mm to (142.4, 110.4), turned to 180 degrees
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Connections:
- C116 pad 1: Net-(U16-FB) -> +3V3
- L2 pad 2: Net-(U16-FB) -> +3V3
- R106 pad 1: GND -> +3V3
- R106 pad 2: Net-(U15-~{ENABLE}) -> Net-(U15-~{RESET})
- R13 pad 1: GND -> +3V3
- R13 pad 2: Net-(U4-~{ENABLE}) -> Net-(U4-~{RESET})
- R14 pad 1: GND -> +3V3
- R14 pad 2: Net-(U5-~{ENABLE}) -> Net-(U5-~{RESET})
- R22 pad 1: GND -> +3V3
- R22 pad 2: Net-(U6-~{ENABLE}) -> Net-(U6-~{RESET})
- R30 pad 1: GND -> +3V3
- R30 pad 2: Net-(U7-~{ENABLE}) -> Net-(U7-~{RESET})
- R38 pad 1: GND -> +3V3
- R38 pad 2: Net-(U8-~{ENABLE}) -> Net-(U8-~{RESET})
- R46 pad 1: GND -> +3V3
- R46 pad 2: Net-(U9-~{ENABLE}) -> Net-(U9-~{RESET})
- R54 pad 1: GND -> +3V3
- R54 pad 2: Net-(U10-~{ENABLE}) -> Net-(U10-~{RESET})
- R62 pad 1: GND -> +3V3
- R62 pad 2: Net-(U11-~{ENABLE}) -> Net-(U11-~{RESET})
- R79 pad 1: Net-(U16-FB) -> +3V3
- R81 pad 1: GND -> +3V3
- R81 pad 2: Net-(U12-~{ENABLE}) -> Net-(U12-~{RESET})
- R90 pad 1: GND -> +3V3
- R90 pad 2: Net-(U13-~{ENABLE}) -> Net-(U13-~{RESET})
- R98 pad 1: GND -> +3V3
- R98 pad 2: Net-(U14-~{ENABLE}) -> Net-(U14-~{RESET})
- S1 pad 1: +12V -> /In1
- S1 pad 2: Net-(D2-K) -> GND
- S1 pad 3: unconnected-(S1-Pad3) -> /In2
- TP1 pad 1: Net-(U16-FB) -> +3V3
- TP8 pad 1: /RESET_N -> /ENABLE_N
- U1 pad 38: /RESET_N -> /ENABLE_N
- U10 pad 12: /RESET_N -> Net-(U10-~{RESET})
- U10 pad 2: Net-(U10-~{ENABLE}) -> /ENABLE_N
- U11 pad 12: /RESET_N -> Net-(U11-~{RESET})
- U11 pad 2: Net-(U11-~{ENABLE}) -> /ENABLE_N
- U12 pad 12: /RESET_N -> Net-(U12-~{RESET})
- U12 pad 2: Net-(U12-~{ENABLE}) -> /ENABLE_N
- U13 pad 12: /RESET_N -> Net-(U13-~{RESET})
- U13 pad 2: Net-(U13-~{ENABLE}) -> /ENABLE_N
- U14 pad 12: /RESET_N -> Net-(U14-~{RESET})
- U14 pad 2: Net-(U14-~{ENABLE}) -> /ENABLE_N
- U15 pad 12: /RESET_N -> Net-(U15-~{RESET})
- U15 pad 2: Net-(U15-~{ENABLE}) -> /ENABLE_N
- U16 pad 3: Net-(U16-FB) -> +3V3
- U4 pad 12: /RESET_N -> Net-(U4-~{RESET})
- U4 pad 2: Net-(U4-~{ENABLE}) -> /ENABLE_N
- U5 pad 12: /RESET_N -> Net-(U5-~{RESET})
- U5 pad 2: Net-(U5-~{ENABLE}) -> /ENABLE_N
- U6 pad 12: /RESET_N -> Net-(U6-~{RESET})
- U6 pad 2: Net-(U6-~{ENABLE}) -> /ENABLE_N
- U7 pad 12: /RESET_N -> Net-(U7-~{RESET})
- U7 pad 2: Net-(U7-~{ENABLE}) -> /ENABLE_N
- U8 pad 12: /RESET_N -> Net-(U8-~{RESET})
- U8 pad 2: Net-(U8-~{ENABLE}) -> /ENABLE_N
- U9 pad 12: /RESET_N -> Net-(U9-~{RESET})
- U9 pad 2: Net-(U9-~{ENABLE}) -> /ENABLE_N
Routing:
- net /ENABLE_N: track 0.00 -> 505.0 mm, vias 0 -> 4
- net /RESET_N: track 376.9 -> 0.00 mm, vias 3 -> 0
- net GND: track 483.0 -> 432.8 mm, vias 102 -> 87
- net +3V3: track 225.1 -> 257.3 mm, vias 39 -> 56
- net /In2: track 25.1 -> 49.2 mm
- net /In3: track 16.4 -> 40.4 mm
- net /In1: track 34.8 -> 55.2 mm
- net Net-(U16-FB): track 12.5 -> 0.00 mm
- net Net-(U8-~{ENABLE}): track 5.01 -> 0.00 mm
- net Net-(U9-~{ENABLE}): track 5.01 -> 0.00 mm
- net Net-(U7-~{ENABLE}): track 5.01 -> 0.00 mm
- net Net-(U6-~{ENABLE}): track 5.01 -> 0.00 mm
- net Net-(U5-~{ENABLE}): track 5.01 -> 0.00 mm
- net Net-(U4-~{ENABLE}): track 5.01 -> 0.00 mm
- net Net-(U14-~{ENABLE}): track 5.01 -> 0.00 mm
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- added copper zone on F.Cu, net +12V
- added copper zone on F.Cu, net +3V3
- removed copper zone on B.Cu, net +12V
Other:
- board text removed: "1"
- board text removed: "2"
- board text removed: "3"
