File: DST.kicad_sch (KiCad schematic)
At the start: 214 parts, among them J1 1712805, J10 1712805, J11 1712805, J12 1712805, J2 1712805, J3 1712805, J4 1712805, J5 1712805, J6 1712805, J7 1712805, J8 1712805, J9 1712805, SW1 SW_Push, SW2 SW_Push, U1 RP2350B-QFN80, U10 DRIVER-A4988SETTR-T_QFN28_, U11 DRIVER-A4988SETTR-T_QFN28_, U12 DRIVER-A4988SETTR-T_QFN28_, U13 DRIVER-A4988SETTR-T_QFN28_, U14 DRIVER-A4988SETTR-T_QFN28_, U15 DRIVER-A4988SETTR-T_QFN28_, U2 ABM8-272-T3, U3 W25Q128JVSIQ, U4 DRIVER-A4988SETTR-T_QFN28_, U5 DRIVER-A4988SETTR-T_QFN28_, U6 DRIVER-A4988SETTR-T_QFN28_, U7 DRIVER-A4988SETTR-T_QFN28_, U8 DRIVER-A4988SETTR-T_QFN28_, U9 DRIVER-A4988SETTR-T_QFN28_

Commit message: updated kicad files
Parts:
- removed C1, C15, C23, C31, C39, C47, C61, C62, C63, C85, C86, C87: 0.22 µF, symbol Device:C
- removed C10, C12, C13, C16, C20, C21, C24, C28, C29, C32, C36, C37, C40, C44, C45, C48, C5, C52, C53, C54, C55, C56, C57, C64, C65, C66, C76, C77, C78, C79, C80, C81, C88, C89, C9, C90: 0.1 µF, symbol Device:C
- removed C11, C18, C26, C34, C42, C50, C70, C71, C72, C94, C95, C96: 0.1 µF, symbol Device:C_Polarized
- removed C14, C17, C22, C25, C30, C33, C38, C41, C46, C49, C58, C59, C6, C60, C67, C68, C69, C8, C82, C83, C84, C91, C92, C93: 100 µF, symbol Device:C
- removed C19, C27, C35, C43, C51, C7, C73, C74, C75, C97, C98, C99: 100 µF, symbol Device:C_Polarized
- removed J1, J10, J11, J12, J2, J3, J4, J5, J6, J7, J8, J9: 1712805, 1712805:PHOENIX_1712805, symbol 1712805:1712805
- removed R1, R2: R, symbol Device:R
- removed R10, R11, R14, R15, R16, R19, R20, R21, R24, R25, R26, R29, R30, R31, R34, R35, R36, R41, R43, R45, R46, R47, R48, R49, R50, R51, R56, R58, R6, R60, R61, R62, R63, R64, R65, R66, R7: 10k, symbol Device:R
- removed R12, R13, R17, R18, R22, R23, R27, R28, R32, R33, R37, R38, R39, R40, R42, R44, R52, R53, R54, R55, R57, R59, R8, R9: 0.2, symbol Device:R
- removed U10, U11, U12, U13, U14, U15, U4, U5, U6, U7, U8, U9: DRIVER-A4988SETTR-T_QFN28_, DRIVER-A4988SETTR-T_QFN28_:QFN28G_0.5-5X5MM, symbol DRIVER-A4988SETTR-T_QFN28_:DRIVER-A4988SETTR-T_QFN28_
- added C115, C116: 0.1 µF, Capacitor_SMD:C_0603_1608Metric, symbol Device:C_Polarized
- added D1, D2: D_Schottky, SSB43L-E352T:DIOM5436X244N, symbol Device:D_Schottky
- added D3, D4: PTVS3V3D1BALYL, PTVS3V3D1BALYL_REAL:PESD5V0S1BL315, symbol PTVS3V3D1BALYL:PTVS3V3D1BALYL
- added D5, D7: 5988170107F, 5988170107F:LEDC2012X70N, symbol 5988170107F:5988170107F
- added D6: KT-0603R, KT-0603R:LED_KT-0603R, symbol KT-0603R:KT-0603R
- added J1: 1727010, 1727010:PHOENIX_1727010, symbol 1727010:1727010
- added J10, J11, J12, J15, J16, J17, J4, J5, J6, J7, J8, J9: 77311-462K05LF, 77311-462K05LF:HDRV5W62P0X254_1X5_1270X240X1624P, symbol 77311-462K05LF:77311-462K05LF
- added J13: DC-005-5A-2.0, DC-005-5A-2.0:XKB_DC-005-5A-2.0, symbol DC-005-5A-2.0:DC-005-5A-2.0
- added J14: 1981568-1, 1981568-1:TE_1981568-1, symbol 1981568-1:1981568-1
- added J2: 5-146280-3, 5-146280-3:TE_5-146280-3, symbol 5-146280-3:5-146280-3
- added J3: 20021121-00020C4LF, 20021121-00020C4LF:AMPHENOL_20021121-00020C4LF, symbol 20021121-00020C4LF:20021121-00020C4LF
- added L2: 47uH, Inductor_SMD:L_0805_2012Metric, symbol Device:L
- added R73, R74, R75: 10k, Resistor_SMD:R_0402_1005Metric, symbol Device:R
- added R76, R77: DNF, Resistor_SMD:R_0805_2012Metric, symbol Device:R
- added R79: 60, Resistor_SMD:R_0805_2012Metric, symbol Device:R
- added R80: 60, Resistor_SMD:R_0402_1005Metric, symbol Device:R
- added R82: 100, Resistor_SMD:R_0402_1005Metric, symbol Device:R
- added S1: 100SP1T2B4M7QE, 100SP1T2B4M7QE:SW_100SP1T2B4M7QE, symbol 100SP1T2B4M7QE:100SP1T2B4M7QE
- added SW3: 219-3LPSTR, 219-3LPSTR:SW_219-3LPSTR, symbol 219-3LPSTR:219-3LPSTR
- added TP1, TP10, TP11, TP12, TP2, TP3, TP8, TP9: TestPoint, TestPoint:TestPoint_Pad_2.0x2.0mm, symbol Connector:TestPoint
- added U16: PMIC-AP1509-SG-13_SOIC8_, PMIC-AP1509-SG-13_SOIC8_:SOIC8-1.27-5X4MM, symbol PMIC-AP1509-SG-13_SOIC8_:PMIC-AP1509-SG-13_SOIC8_
- C100, C101: value 100n -> 1u; footprint (none) -> Capacitor_SMD:C_0402_1005Metric
- C102, C103: value 100n -> 10n; footprint (none) -> Capacitor_SMD:C_0402_1005Metric
- C104, C105, C106, C107, C108, C109, C110, C111, C112, C113, C114, C2, C4: footprint (none) -> Capacitor_SMD:C_0402_1005Metric
- C3: value C -> 100n; footprint (none) -> Capacitor_SMD:C_0402_1005Metric
- L1: footprint (none) -> Inductor_SMD:L_0402_1005Metric
- R3: value R -> 0; footprint (none) -> Resistor_SMD:R_0805_2012Metric
- R4, R5: value R -> 1k; footprint (none) -> Resistor_SMD:R_0805_2012Metric
- R67, R68: value R -> 27; footprint (none) -> Resistor_SMD:R_0402_1005Metric
- R69: footprint (none) -> Resistor_SMD:R_0805_2012Metric
- R70: value R -> 33; footprint (none) -> Resistor_SMD:R_0805_2012Metric
- SW1, SW2: footprint (none) -> SPEH110101:SPEH110101
- U1: footprint (none) -> Package_DFN_QFN:QFN-80-1EP_10x10mm_P0.4mm_EP3.4x3.4mm_ThermalVias
- U2: footprint ABM8-272-T3:ABM8-272-T3 -> ABM8:ABM8-272-T3
Connections:
- net DIR1: now also U1.79 (GPIO2), TP3.1; no longer U1.78 (GPIO1)
- net DIR10: now also U1.20 (GPIO20); no longer U1.19 (GPIO19)
- net DIR11: now also U1.22 (GPIO22); no longer U1.21 (GPIO21)
- net DIR12: now also U1.25 (GPIO24); no longer U1.23 (GPIO23)
- net DIR2: now also U1.1 (GPIO4); no longer U1.80 (GPIO3)
- net DIR3: now also U1.3 (GPIO6); no longer U1.2 (GPIO5)
- net DIR4: now also U1.6 (GPIO8); no longer U1.4 (GPIO7)
- net DIR5: now also U1.8 (GPIO10); no longer U1.7 (GPIO9)
- net DIR6: now also U1.11 (GPIO12); no longer U1.9 (GPIO11)
- net DIR7: now also U1.13 (GPIO14); no longer U1.12 (GPIO13)
- net DIR8: now also U1.16 (GPIO16); no longer U1.14 (GPIO15)
- net DIR9: now also U1.18 (GPIO18); no longer U1.17 (GPIO17)
- net GND: now also C115.2, C116.2, D1.2 (A), D3.2 (K2), D4.2 (K2), D5.C, D6.C, D7.C, J1.02, J13.2, J14.5, J2.2, SW3.1_1, SW3.2_1, SW3.3_1, U16.4 (SD), U16.5 (GND), U16.6 (GND@1), U16.7 (GND@2), U16.8 (GND@3)
- net GPIO0: now also U1.77 (GPIO0), R76.1
- net OUT1A1: now also J4.1, TP9.1
- net OUT1A10: now also J11.1
- net OUT1A11: now also J15.1
- net OUT1A12: now also J17.1
- net OUT1A2: now also J6.1
- net OUT1A3: now also J8.1
- net OUT1A4: now also J10.1
- net OUT1A5: now also J12.1
- net OUT1A6: now also J16.1
- net OUT1A7: now also J5.1
- net OUT1A8: now also J7.1
- net OUT1A9: now also J9.1
- net OUT1B1: now also J4.2, TP10.1
- net OUT1B10: now also J11.2
- net OUT1B11: now also J15.2
- net OUT1B12: now also J17.2
- net OUT1B2: now also J6.2
- net OUT1B3: now also J8.2
- net OUT1B4: now also J10.2
- net OUT1B5: now also J12.2
- net OUT1B6: now also J16.2
- net OUT1B7: now also J5.2
- net OUT1B8: now also J7.2
- net OUT1B9: now also J9.2
- net OUT2A1: now also J4.3, TP11.1
- net OUT2A10: now also J11.3
- net OUT2A11: now also J15.3
- net OUT2A12: now also J17.3
- net OUT2A2: now also J6.3
- net OUT2A3: now also J8.3
- net OUT2A4: now also J10.3
- net OUT2A5: now also J12.3
- net OUT2A6: now also J16.3
- net OUT2A7: now also J5.3
- net OUT2A8: now also J7.3
- net OUT2A9: now also J9.3
- net OUT2B1: now also J4.4, TP12.1
- net OUT2B10: now also J11.4
- net OUT2B11: now also J15.4
- net OUT2B12: now also J17.4
- net OUT2B2: now also J6.4
- net OUT2B3: now also J8.4
- net OUT2B4: now also J10.4
- net OUT2B5: now also J12.4
- net OUT2B6: now also J16.4
- net OUT2B7: now also J5.4
- net OUT2B8: now also J7.4
- net OUT2B9: now also J9.4
- net QSPI_SCLK: now also U3.6 (CLK); no longer U3.7 (/HOLD/RESET(IO3))
- net QSPI_SD0: now also U3.5 (DI(IO0)); no longer U3.6 (CLK)
- net QSPI_SD1: now also U3.2 (DO(IO1)); no longer U3.5 (DI(IO0))
- net QSPI_SD2: now also U3.3 (/WP(IO2)); no longer U3.2 (DO(IO1))
- net QSPI_SD3: now also U3.7 (/HOLD/RESET(IO3)); no longer U3.3 (/WP(IO2))
- net STEP1: now also U1.78 (GPIO1), TP2.1; no longer U1.77 (GPIO0)
- net STEP10: now also U1.19 (GPIO19); no longer U1.18 (GPIO18)
- net STEP11: now also U1.21 (GPIO21); no longer U1.20 (GPIO20)
- net STEP12: now also U1.23 (GPIO23); no longer U1.22 (GPIO22)
- net STEP2: now also U1.80 (GPIO3); no longer U1.79 (GPIO2)
- net STEP3: now also U1.2 (GPIO5); no longer U1.1 (GPIO4)
- net STEP4: now also U1.4 (GPIO7); no longer U1.3 (GPIO6)
- net STEP5: now also U1.7 (GPIO9); no longer U1.6 (GPIO8)
- net STEP6: now also U1.9 (GPIO11); no longer U1.8 (GPIO10)
- net STEP7: now also U1.12 (GPIO13); no longer U1.11 (GPIO12)
- net STEP8: now also U1.14 (GPIO15); no longer U1.13 (GPIO14)
- net STEP9: now also U1.17 (GPIO17); no longer U1.16 (GPIO16)
- net SWCLK: now also J2.1
- net SWD: now also J2.3
- net USB_D+: now also D4.1 (K1), J14.3, J3.18
- net USB_D-: now also D3.1 (K1), J14.2, J3.20
- net at R3.2, U3.1 (/CS): now also R76.2, R77.1
- net In1: now reaches U1.26 (GPIO25)
- net In1: now also R73.1, SW3.1
- net In2: now reaches U1.27 (GPIO26)
- net In2: now also R74.1, SW3.2
- net In3: now reaches U1.28 (GPIO27)
- net In3: now also R75.1, SW3.3
- net at U1.36 (GPIO28): now also R80.1
- net at U1.37 (GPIO29): now also R82.1
- net RESET_N: now reaches U1.38 (GPIO30)
- net RESET_N: now also TP8.1
- net EXT_GPIO1: now reaches U1.39 (GPIO31)
- net EXT_GPIO1: now also J3.3
- net EXT_GPIO2: now reaches U1.40 (GPIO32)
- net EXT_GPIO2: now also J3.5
- net EXT_GPIO3: now reaches U1.42 (GPIO33)
- net EXT_GPIO3: now also J3.7
- net EXT_GPIO4: now reaches U1.43 (GPIO34)
- net EXT_GPIO4: now also J3.9
- net EXT_GPIO5: now reaches U1.44 (GPIO35)
- net EXT_GPIO5: now also J3.11
- net EXT_GPIO6: now reaches U1.45 (GPIO36)
- net EXT_GPIO6: now also J3.13
- net EXT_GPIO7: now reaches U1.46 (GPIO37)
- net EXT_GPIO7: now also J3.15
- net EXT_GPIO8: now reaches U1.47 (GPIO38)
- net EXT_GPIO8: now also J3.17
- net EXT_GPIO9: now reaches U1.48 (GPIO39)
- net EXT_GPIO9: now also J3.19
- net EXT_GPIO10: now reaches U1.49 (GPIO40_ADC0)
- net EXT_GPIO10: now also J3.2
- net EXT_GPIO11: now reaches U1.52 (GPIO41_ADC1)
- net EXT_GPIO11: now also J3.4
- net EXT_GPIO12: now reaches U1.53 (GPIO42_ADC2)
- net EXT_GPIO12: now also J3.6
- net EXT_GPIO13: now reaches U1.54 (GPIO43_ADC3)
- net EXT_GPIO13: now also J3.8
- net EXT_GPIO14: now reaches U1.55 (GPIO44_ADC4)
- net EXT_GPIO14: now also J3.10
- net EXT_GPIO15: now reaches U1.56 (GPIO45_ADC5)
- net EXT_GPIO15: now also J3.12
- net EXT_GPIO16: now reaches U1.57 (GPIO46_ADC6)
- net EXT_GPIO16: now also J3.14
- net EXT_GPIO17: now reaches U1.58 (GPIO47_ADC7)
- net EXT_GPIO17: now also J3.16
- net +3.3V renamed +3V3
- net +3V3: now also J10.5, J11.5, J12.5, J15.5, J16.5, J17.5, J4.5, J5.5, J6.5, J7.5, J8.5, J9.5, R73.2, R74.2, R75.2, R77.2
- new net: D6.A, R82.2
- new net: D2.1 (K), S1.2
- new net: D5.A, R80.2
- new net: D1.1 (K), L2.1, U16.2 (OUTPUT)
- new net: C116.1, L2.2, R79.1, TP1.1, U16.3 (FB)
- new net: J14.SH1 (SHIELD), J14.SH2 (SHIELD), J14.SH3 (SHIELD), J14.SH4 (SHIELD), J14.SH5 (SHIELD), J14.SH6 (SHIELD)
- new net: D7.A, R79.2
- new net +12V: C115.1, S1.1, U16.1 (VIN)
- new net 12V_IN: D2.2 (A), J1.01, J13.1
- new net EXT_GPIO0: J3.1
- no-connect marks 0 -> 5
Other:
- added sheet MotorDriver1 (untitled.kicad_sch)
- added sheet MotorDriver10 (untitled.kicad_sch)
- added sheet MotorDriver11 (untitled.kicad_sch)
- added sheet MotorDriver12 (untitled.kicad_sch)
- added sheet MotorDriver2 (untitled.kicad_sch)
- added sheet MotorDriver3 (untitled.kicad_sch)
- added sheet MotorDriver4 (untitled.kicad_sch)
- added sheet MotorDriver5 (untitled.kicad_sch)
- added sheet MotorDriver6 (untitled.kicad_sch)
- added sheet MotorDriver7 (untitled.kicad_sch)
- added sheet MotorDriver8 (untitled.kicad_sch)
- added sheet MotorDriver9 (untitled.kicad_sch)
- note added: "5988170107F GREEN LED"
- note added: "Double barrel power input Pin 3 does not need to be connected as its used for swtiching"
- note added: "Flash memory"
- note added: "Green LED 5988170107F"
- note added: "KT-0603R RED LED"
- note added: "Micro USB B input"
- note added: "Occilator"
- note added: "Output Header Pins"
- note added: "Toggle switches to control functionality"
- note added: "backup power input"
- moved on the sheet: R4, SW1

Commit message: newsest changes
Parts:
- removed D5, D7: 5988170107F, 5988170107F:LEDC2012X70N, symbol 5988170107F:5988170107F
- removed S1: 100SP1T2B4M7QE, 100SP1T2B4M7QE:SW_100SP1T2B4M7QE, symbol 100SP1T2B4M7QE:100SP1T2B4M7QE
- removed SW3: 219-3LPSTR, 219-3LPSTR:SW_219-3LPSTR, symbol 219-3LPSTR:219-3LPSTR
- added LED1, LED2: 150080GS75000, KiCad:LEDM2012X80N, symbol 150080GS75000:150080GS75000
- added S1: NDS-03V, NDS-03V:NDS03V, symbol NDS-03V:NDS-03V
- added S2: 1MS3T1B1M2QES, 1MS3T1B1M2QES, symbol 1MS3T1B1M2QES:1MS3T1B1M2QES
Connections:
- net +12V: now also S2.2 (COMM)
- net +3V3: now also C116.1, L2.2, R79.1, TP1.1, U16.3 (FB)
- net GND: now also LED1.2 (A), LED2.2 (A), S1.2 (N.O._1), S1.4 (N.O._2), S1.6 (N.O._3)
- net In1: now also S1.1 (COM_1)
- net In2: now also S1.3 (COM_2)
- net In3: now also S1.5 (COM_3)
- net at D2.1 (K): now also S2.1 (NO)
- net at R80.2: now also LED1.1 (K)
- net at R79.2: now also LED2.1 (K)
- net RESET_N renamed ENABLE_N
Other:
- sheet MotorDriver1 ports: added ENABLE_N; removed RESET_N
- sheet MotorDriver10 ports: added ENABLE_N; removed RESET_N
- sheet MotorDriver11 ports: added ENABLE_N; removed RESET_N
- sheet MotorDriver12 ports: added ENABLE_N; removed RESET_N
- sheet MotorDriver2 ports: added ENABLE_N; removed RESET_N
- sheet MotorDriver3 ports: added ENABLE_N; removed RESET_N
- sheet MotorDriver4 ports: added ENABLE_N; removed RESET_N
- sheet MotorDriver5 ports: added ENABLE_N; removed RESET_N
- sheet MotorDriver6 ports: added ENABLE_N; removed RESET_N
- sheet MotorDriver7 ports: added ENABLE_N; removed RESET_N
- sheet MotorDriver8 ports: added ENABLE_N; removed RESET_N
- sheet MotorDriver9 ports: added ENABLE_N; removed RESET_N
- moved on the sheet: D2
