File: untitled.kicad_sch (KiCad schematic)
At the start: 17 parts, among them U4 DRIVER-A4988SETTR-T_QFN28_

Commit message: newsest changes
Connections:
- net RESET_N is gone; now on an unnamed net: U4.12 (~{RESET})
- net +3V3: now also R13.1
- net GND: no longer R13.1
- net at R13.2: no longer U4.2 (~{ENABLE})
- new net ENABLE_N: U4.2 (~{ENABLE})
Other:
- moved on the sheet: R13
Changed lines of the file:
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@@
 	(wire
 		(pts
-			(xy 104.14 85.09) (xy 104.14 86.36)
-		)
-		(stroke
-			(width 0)
-			(type default)
-		)
-	)
-	(wire
-		(pts
 			(xy 179.07 91.44) (xy 179.07 93.98)
 		)
@@
 	(wire
 		(pts
-			(xy 104.14 86.36) (xy 106.68 86.36)
+			(xy 127 111.76) (xy 127 116.84)
 		)
 		(stroke
@@
 	(wire
 		(pts
-			(xy 127 111.76) (xy 127 116.84)
+			(xy 104.14 83.82) (xy 106.68 83.82)
 		)
 		(stroke
@@
 	(wire
 		(pts
-			(xy 104.14 83.82) (xy 106.68 83.82)
+			(xy 165.1 93.98) (xy 166.37 93.98)
 		)
 		(stroke
@@
 	(wire
 		(pts
-			(xy 165.1 93.98) (xy 166.37 93.98)
+			(xy 95.25 86.36) (xy 106.68 86.36)
 		)
 		(stroke
@@
 	(wire
 		(pts
-			(xy 102.87 85.09) (xy 104.14 85.09)
-		)
-		(stroke
-			(width 0)
-			(type default)
-		)
-	)
-	(wire
-		(pts
 			(xy 140.97 114.3) (xy 134.62 114.3)
 		)
@@
 	(wire
 		(pts
-			(xy 90.17 85.09) (xy 95.25 85.09)
-		)
-		(stroke
-			(width 0)
-			(type default)
-		)
-	)
-	(wire
-		(pts
 			(xy 132.08 115.57) (xy 132.08 111.76)
 		)
@@
 	(wire
 		(pts
-			(xy 129.54 111.76) (xy 129.54 118.11)
+			(xy 129.54 111.76) (xy 129.54 128.27)
 		)
 		(stroke
@@
 	(wire
 		(pts
-			(xy 140.97 121.92) (xy 140.97 124.46)
+			(xy 140.97 121.92) (xy 140.97 127)
 		)
 		(stroke
@@
 	(wire
 		(pts
+			(xy 129.54 135.89) (xy 129.54 143.51)
+		)
+		(stroke
+			(width 0)
+			(type default)
+		)
+	)
+	(wire
+		(pts
 			(xy 124.46 67.31) (xy 124.46 71.12)
 		)
@@
 	(wire
 		(pts
+			(xy 129.54 143.51) (xy 130.81 143.51)
+		)
+		(stroke
+			(width 0)
+			(type default)
+		)
+	)
+	(wire
+		(pts
 			(xy 147.32 93.98) (xy 165.1 93.98)
 		)
@@
 		)
 	)
+	(hierarchical_label "ENABLE_N"
+		(shape input)
+		(at 95.25 86.36 180)
+		(effects
+			(font
+				(size 0.762 0.762)
+			)
+			(justify right)
+		)
+	)
 	(hierarchical_label "STEP"
 		(shape input)
@@
 		)
 	)
-	(hierarchical_label "RESET_N"
-		(shape input)
-		(at 129.54 118.11 270)
-		(effects
-			(font
-				(size 0.762 0.762)
-			)
-			(justify right)
-		)
-	)
 	(symbol
 		(lib_id "Device:R")
@@
 	)
 	(symbol
+		(lib_id "power:+3V3")
+		(at 130.81 143.51 270)
+		(unit 1)
+		(exclude_from_sim no)
+		(in_bom yes)
+		(on_board yes)
+		(dnp no)
+		(fields_autoplaced yes)
+		(property "Reference" "#PWR0216"
+			(at 127 143.51 0)
+			(effects
+				(font
+					(size 1.27 1.27)
+				)
+				(hide yes)
+			)
+		)
+		(property "Value" "+3V3"
+			(at 134.62 143.5099 90)
+			(effects
+				(font
+					(size 1.27 1.27)
+				)
+				(justify left)
+			)
+		)
+		(property "Footprint" ""
+			(at 130.81 143.51 0)
+			(effects
+				(font
+					(size 1.27 1.27)
+				)
+				(hide yes)
+			)
+		)
+		(property "Datasheet" ""
+			(at 130.81 143.51 0)
+			(effects
+				(font
+					(size 1.27 1.27)
+				)
+				(hide yes)
+			)
+		)
+		(property "Description" "Power symbol creates a global label with name \"+3V3\""
+			(at 130.81 143.51 0)
+			(effects
+				(font
+					(size 1.27 1.27)
+				)
+				(hide yes)
+			)
+		)
+		(pin "1"
+		)
+		(instances
+			(project "DST"
+				(path "/cf4d8f46-3b3e-4ef2-a306-bbe888c527c6/0715f16f-576a-41e7-857e-915f3aa7cbb3"
+					(reference "#PWR0223")
+					(unit 1)
+				)
+				(path "/cf4d8f46-3b3e-4ef2-a306-bbe888c527c6/3903b079-1378-4ce9-b008-c916781b3188"
+					(reference "#PWR0218")
+					(unit 1)
+				)
+				(path "/cf4d8f46-3b3e-4ef2-a306-bbe888c527c6/5c1e5e7a-8ccb-4de2-a3bc-3f7352ee623b"
+					(reference "#PWR0217")
+					(unit 1)
+				)
+				(path "/cf4d8f46-3b3e-4ef2-a306-bbe888c527c6/7205875f-0bab-4f88-928e-9aa70b3abf32"
+					(reference "#PWR0225")
+					(unit 1)
+				)
+				(path "/cf4d8f46-3b3e-4ef2-a306-bbe888c527c6/76029fa4-aa94-4169-b97c-0f498e8af583"
+					(reference "#PWR0219")
+					(unit 1)
+				)
+				(path "/cf4d8f46-3b3e-4ef2-a306-bbe888c527c6/77d91239-2fe8-4810-a8b1-8fe25dfb81bc"
+					(reference "#PWR0222")
+					(unit 1)
+				)
+				(path "/cf4d8f46-3b3e-4ef2-a306-bbe888c527c6/986292b7-1f07-4573-97c1-fe4afc788d80"
+					(reference "#PWR0226")
+					(unit 1)
+				)
+				(path "/cf4d8f46-3b3e-4ef2-a306-bbe888c527c6/a30b9f38-db07-4da1-810c-dda9441ad49a"
+					(reference "#PWR0227")
+					(unit 1)
+				)
+				(path "/cf4d8f46-3b3e-4ef2-a306-bbe888c527c6/b2a66a53-739c-40f5-8de8-8cbc212c4b3e"
+					(reference "#PWR0220")
+					(unit 1)
+				)
+				(path "/cf4d8f46-3b3e-4ef2-a306-bbe888c527c6/b839523b-062b-41ca-b392-573d8460955d"
+					(reference "#PWR0224")
+					(unit 1)
+				)
+				(path "/cf4d8f46-3b3e-4ef2-a306-bbe888c527c6/f0501b55-b009-4cb3-8d90-8ba3daaff44e"
+					(reference "#PWR0221")
+					(unit 1)
+				)
+				(path "/cf4d8f46-3b3e-4ef2-a306-bbe888c527c6/ff1eb6d5-9192-4009-b7a2-a19bd13ed29b"
+					(reference "#PWR0216")
+					(unit 1)
+				)
+			)
+		)
+	)
+	(symbol
 		(lib_id "power:GND")
 		(at 171.45 74.93 0)
@@
 	(symbol
 		(lib_id "power:+3V3")
-		(at 140.97 124.46 180)
+		(at 140.97 127 270)
 		(unit 1)
 		(exclude_from_sim no)
@@
 		(on_board yes)
 		(dnp no)
-		(fields_autoplaced yes)
 		(property "Reference" "#PWR0169"
-			(at 140.97 120.65 0)
+			(at 137.16 127 0)
 			(effects
 				(font
@@
 		)
 		(property "Value" "+3V3"
-			(at 140.9701 128.27 90)
+			(at 144.78 126.9999 90)
 			(effects
 				(font
@@
 		)
 		(property "Footprint" ""
-			(at 140.97 124.46 0)
+			(at 140.97 127 0)
 			(effects
 				(font
@@
 		)
 		(property "Datasheet" ""
-			(at 140.97 124.46 0)
+			(at 140.97 127 0)
 			(effects
 				(font
@@
 		)
 		(property "Description" "Power symbol creates a global label with name \"+3V3\""
-			(at 140.97 124.46 0)
+			(at 140.97 127 0)
 			(effects
 				(font
@@
 	(symbol
 		(lib_id "Device:R")
-		(at 99.06 85.09 90)
+		(at 129.54 132.08 180)
 		(unit 1)
 		(exclude_from_sim no)
@@
 		(dnp no)
 		(property "Reference" "R13"
-			(at 99.314 80.518 90)
+			(at 124.968 131.826 90)
 			(effects
 				(font
@@
 		)
 		(property "Value" "10k"
-			(at 98.552 82.804 90)
+			(at 127.254 132.588 90)
 			(effects
 				(font
@@
 		)
 		(property "Footprint" "Resistor_SMD:R_0805_2012Metric"
-			(at 99.06 86.868 90)
+			(at 131.318 132.08 90)
 			(effects
 				(font
@@
 		)
 		(property "Datasheet" "~"
-			(at 99.06 85.09 0)
+			(at 129.54 132.08 0)
 			(effects
 				(font
@@
 		)
 		(property "Description" "Resistor"
-			(at 99.06 85.09 0)
+			(at 129.54 132.08 0)
 			(effects
 				(font
@@
 					(unit 1)
 				)
-			)
-		)
-	)
-	(symbol
-		(lib_id "power:GND")
-		(at 90.17 85.09 0)
-		(unit 1)
-		(exclude_from_sim no)
-		(in_bom yes)
-		(on_board yes)
-		(dnp no)
-		(fields_autoplaced yes)
-		(property "Reference" "#PWR0216"
-			(at 90.17 91.44 0)
-			(effects
-				(font
-					(size 1.27 1.27)
-				)
-				(hide yes)
-			)
-		)
-		(property "Value" "GND"
-			(at 90.17 90.17 0)
-			(effects
-				(font
-					(size 1.27 1.27)
-				)
-			)
-		)
-		(property "Footprint" ""
-			(at 90.17 85.09 0)
-			(effects
-				(font
-					(size 1.27 1.27)
-				)
-				(hide yes)
-			)
-		)
-		(property "Datasheet" ""
-			(at 90.17 85.09 0)
-			(effects
-				(font
-					(size 1.27 1.27)
-				)
-				(hide yes)
-			)
-		)
-		(property "Description" "Power symbol creates a global label with name \"GND\" , ground"
-			(at 90.17 85.09 0)
-			(effects
-				(font
-					(size 1.27 1.27)
-				)
-				(hide yes)
-			)
-		)
-		(pin "1"
-		)
-		(instances
-			(project "DST"
-				(path "/cf4d8f46-3b3e-4ef2-a306-bbe888c527c6/0715f16f-576a-41e7-857e-915f3aa7cbb3"
-					(reference "#PWR0223")
-					(unit 1)
-				)
-				(path "/cf4d8f46-3b3e-4ef2-a306-bbe888c527c6/3903b079-1378-4ce9-b008-c916781b3188"
-					(reference "#PWR0218")
-					(unit 1)
-				)
-				(path "/cf4d8f46-3b3e-4ef2-a306-bbe888c527c6/5c1e5e7a-8ccb-4de2-a3bc-3f7352ee623b"
-					(reference "#PWR0217")
-					(unit 1)
-				)
-				(path "/cf4d8f46-3b3e-4ef2-a306-bbe888c527c6/7205875f-0bab-4f88-928e-9aa70b3abf32"
-					(reference "#PWR0225")
-					(unit 1)
-				)
-				(path "/cf4d8f46-3b3e-4ef2-a306-bbe888c527c6/76029fa4-aa94-4169-b97c-0f498e8af583"
-					(reference "#PWR0219")
-					(unit 1)
-				)
-				(path "/cf4d8f46-3b3e-4ef2-a306-bbe888c527c6/77d91239-2fe8-4810-a8b1-8fe25dfb81bc"
-					(reference "#PWR0222")
-					(unit 1)
-				)
-				(path "/cf4d8f46-3b3e-4ef2-a306-bbe888c527c6/986292b7-1f07-4573-97c1-fe4afc788d80"
-					(reference "#PWR0226")
-					(unit 1)
-				)
-				(path "/cf4d8f46-3b3e-4ef2-a306-bbe888c527c6/a30b9f38-db07-4da1-810c-dda9441ad49a"
-					(reference "#PWR0227")
-					(unit 1)
-				)
-				(path "/cf4d8f46-3b3e-4ef2-a306-bbe888c527c6/b2a66a53-739c-40f5-8de8-8cbc212c4b3e"
-					(reference "#PWR0220")
-					(unit 1)
-				)
-				(path "/cf4d8f46-3b3e-4ef2-a306-bbe888c527c6/b839523b-062b-41ca-b392-573d8460955d"
-					(reference "#PWR0224")
-					(unit 1)
-				)
-				(path "/cf4d8f46-3b3e-4ef2-a306-bbe888c527c6/f0501b55-b009-4cb3-8d90-8ba3daaff44e"
-					(reference "#PWR0221")
-					(unit 1)
-				)
-				(path "/cf4d8f46-3b3e-4ef2-a306-bbe888c527c6/ff1eb6d5-9192-4009-b7a2-a19bd13ed29b"
-					(reference "#PWR0216")
-					(unit 1)
-				)
